File: hardware/pcbs/control/Control.kicad_pcb (KiCad board)
At the start: 2 copper layers, 71 x 60 mm, 28 parts, among them J1 USB_B, J10 JST PH, J11 Conn_01x02, J2 RJ45_LED_Shielded, J3 RJ45_LED_Shielded, J4 Conn_01x07, J5 Conn_01x07, J6 JST PH, J7 JST PH, J8 JST PH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

Commit message: updated README, split covers
Other:
- board text added: "| Control |"
- board text removed: "| Center |"
